Commit message: fix(description): restore lidar geometry and SO-101 deck

File: src/mentorpi_description/urdf/mecanum.xacro (robot description, xacro)
@@ -96,5 +96,5 @@
     <origin xyz="-0.054 0 0.05" rpy="0 0 0"/>
   </joint>
-  <!-- ===== Camera (AprilTag hand-eye calibrated 2026-07-12) ===== -->
+  <!-- ===== Camera (external transform pending recalibration) ===== -->
   <link name="camera_link">
     <inertial>
@@ -106,5 +106,6 @@
          camera_link 是标定出的光学中心——彩色镜头偏离机身中心 ~3cm(y),
          位于前脸(x)、中高(z)。不加偏移时机身网格会整体跟着光学系平移,
-         看起来"装歪"。标定值本身经地面点云验证,勿动 camera_joint。 -->
+         看起来"装歪"。此机身内参式偏移仍有效；但云台已拆除，下面的
+         camera_joint 是旧安装方式的历史值，最终固定后必须重标。 -->
     <visual>
       <origin rpy="0 0 0" xyz="-0.0137 -0.0305 0.013"/>
@@ -120,5 +121,6 @@
     <parent link="base_link"/>
     <child link="camera_link"/>
-    <!-- AprilTag hand-eye calibration, 2026-07-17; z is ruler-fixed. -->
+    <!-- STALE: AprilTag hand-eye calibration from the removed 2-DOF gimbal,
+         2026-07-17. Keep only as provenance until the direct mount is final. -->
     <origin xyz="0.1114 0.0305 0.0950" rpy="-0.0164 -0.1302 0.0147"/>
   </joint>
@@ -158,49 +160,18 @@
     <parent link="base_link"/>
     <child link="laser_frame"/>
-    <!-- x: ruler-measured 1.4cm behind base center; y: laterally centered;
-         z: measured. RPY (mounting yaw) still to be refined via wall line-fit.
-         装臂(with_so101)不改变雷达高度——臂占据的后向扇区由 laser_filters
-         角度掩膜滤除(见 base.launch.py),现有 2D/3D 地图资产保持有效。 -->
-    <origin xyz="-0.014 0 0.18" rpy="0 0 0"/>
-  </joint>
-  <!-- 雷达塔架(纯外观): base_link.STL 不含塔架,雷达头会悬浮在顶板上方
-       ~9cm。4 根立柱位置 = Codex 网格分析推测的后部 Ø4.3 孔位,与实物
-       待卡尺核对(P0);画出来只为骨架可读,不参与任何 TF/碰撞。 -->
-  <xacro:macro name="lidar_post" params="x y">
-    <visual>
-      <origin xyz="${x} ${y} 0.10125" rpy="0 0 0"/>
-      <geometry><cylinder radius="0.004" length="0.0875"/></geometry>
-      <material name="black"/>
-    </visual>
-  </xacro:macro>
-  <link name="lidar_mount_visual_link">
-    <xacro:lidar_post x="-0.0509" y=" 0.0244"/>
-    <xacro:lidar_post x="-0.0509" y="-0.0244"/>
-    <xacro:lidar_post x="-0.0309" y=" 0.0244"/>
-    <xacro:lidar_post x="-0.0309" y="-0.0244"/>
-    <!-- 相机云台舵机塔(纯外观): 网格切片实测底盘鼻部是台阶状——顶板
-         (z=0.0575)只到 x≈+0.017,前方是 z≈0.0253 的中层甲板(到 x≈0.08)。
-         2-DOF 云台从中层甲板(0.0253)撑到相机机身底(0.0772),高 52mm,
-         不在任何厂商网格里。 -->
-    <visual>
-      <origin xyz="0.088 0 0.0513" rpy="0 0 0"/>
-      <geometry><box size="0.028 0.040 0.052"/></geometry>
-      <material name="black"/>
-    </visual>
-  </link>
-  <joint name="lidar_mount_visual_joint" type="fixed">
-    <parent link="base_link"/>
-    <child link="lidar_mount_visual_link"/>
-    <origin xyz="0 0 0" rpy="0 0 0"/>
+    <!-- Recovered vendor-CAD transform from mecanum.pre_calibration.xacro.
+         base_link is 50.5 mm above ground; lidar_Link.STL spans z=-35..0 mm.
+         This places both the chassis top and lidar bottom at 108.001 mm and
+         laser_frame at 143.001 mm above ground: direct mount, no tower. -->
+    <origin xyz="-0.012242 0 0.092501" rpy="0 0 0"/>
   </joint>
   <!-- ===== SO-101 机械臂(可选, with_so101:=true) =====
-       布局 v2(2026-07-18, 取代 Codex 朝后+riser 方案):
+       布局 v3(2026-07-19, STL/实物测量闭环):
        - 臂朝前(yaw 0): Gemini 2L 天然成为 VLA context 相机,前伸时夹爪入画
-       - 雷达不动: 保住已建地图与低障碍探测;臂收拢姿态占据的后向扇区
+       - 雷达直接贴装于顶板,laser_frame z=0.092501;臂收拢姿态占据的后向扇区
          用激光角度掩膜滤除;抓取作业时停车(motion primitive 安全模型)
        - 臂基座后移至 x=-0.155: 真网格 pan 全程(±110°)扫掠最差裕量
-         头部 23.1mm / 推测立柱 11.4mm(v2_pan.py, 2026-07-18);甲板从
-         共用锚点向后悬伸 ~92mm,SO-101 越过雷达头上方前伸作业
-       - 甲板 deck 为占位 box,P2 CAD 出真实网格后替换 -->
+         头部 36.2mm(恢复 TF 后实算);甲板用雷达后方 4 个 M4 通孔向后悬伸
+         ~92mm,前缘 x=-0.050,与雷达网格保留约 11mm 平面间隙 -->
   <xacro:if value="$(arg with_so101)">
     <xacro:include filename="$(find mentorpi_description)/urdf/so101.xacro"/>
@@ -210,14 +181,14 @@
       mount_rpy="0 0 0"/>
     <!-- 悬伸甲板 (mechanical/printable/so101_deck_plate.py):
-         x -0.195..-0.015, y ±0.048, 顶面 z=0.0655, 底面纵肋 15 深 -->
+         x -0.195..-0.050, y ±0.048, 顶面 z=0.0655, 底面纵肋 15 深 -->
     <link name="so101_deck_link">
       <inertial>
-        <origin xyz="-0.105 0 -0.004" rpy="0 0 0"/>
-        <mass value="0.19"/>
-        <inertia ixx="0.000147" ixy="0" ixz="0"
-                 iyy="0.000515" iyz="0" izz="0.000659"/>
-      </inertial>
-      <visual>
-        <origin xyz="-0.105 0 -0.008" rpy="0 0 0"/>
+        <origin xyz="-0.1225 0 -0.004" rpy="0 0 0"/>
+        <mass value="0.16"/>
+        <inertia ixx="0.000124" ixy="0" ixz="0"
+                 iyy="0.000281" iyz="0" izz="0.000403"/>
+      </inertial>
+      <visual>
+        <origin xyz="-0.1225 0 -0.008" rpy="0 0 0"/>
         <geometry>
           <mesh filename="package://mentorpi_description/meshes/accessories/so101_deck_plate.stl"
@@ -227,6 +198,6 @@
       </visual>
       <collision>
-        <origin xyz="-0.105 0 -0.004" rpy="0 0 0"/>
-        <geometry><box size="0.180 0.096 0.008"/></geometry>
+        <origin xyz="-0.1225 0 -0.004" rpy="0 0 0"/>
+        <geometry><box size="0.145 0.096 0.008"/></geometry>
       </collision>
     </link>

File: src/mentorpi_description/urdf/mentorpi_so101.urdf (robot description, URDF)
Before this commit: robot mentorpi, 23 links, 22 joints
Links:
- removed link lidar_mount_visual_link
- link so101_deck_link: mass 0.19 -> 0.16; geometry collision box size=0.145 0.096 0.008; visual mesh filename=package://mentorpi_description/meshes/accessories/so101_dec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 scale=0.001 0.001 0.001
Joints:
- removed joint lidar_mount_visual_joint
- joint laser_joint: origin xyz=-0.014 0 0.18 rpy=0 0 0 -> xyz=-0.012242 0 0.092501 rpy=0 0 0

File: src/mentorpi_description/urdf/mentorpi_so101.viewer.urdf (robot description, URDF)
Before this commit: robot mentorpi, 23 links, 22 joints
Links:
- removed link lidar_mount_visual_link
- link so101_deck_link: mass 0.19 -> 0.16
Joints:
- removed joint lidar_mount_visual_joint
- joint laser_joint: origin xyz=-0.014 0 0.18 rpy=0 0 0 -> xyz=-0.012242 0 0.092501 rpy=0 0 0
