Commit message: TF source of truth -> URDF: robot_state_publisher + calib write-back
- base.launch.py: replace 3 static_transform_publisher nodes with
  robot_state_publisher rendering mentorpi.xacro runtime_mode:=true
  (omits base_footprint and Orbbec-owned optical frames), plus
  joint_state_publisher for the encoder-less continuous wheel joints
- mecanum.xacro: runtime_mode arg; camera_joint carries the 2026-07-12
  AprilTag hand-eye extrinsic; imu/laser joints match deployed values
- calibrate_camera_extrinsic.py: --update-xacro atomic write-back of
  camera_joint (RMS gate, XML validation, provenance date refresh)
- docs/CLAUDE/TODO: point calibration flow at xacro joints; new TODO
  for laser_joint x/y survey; check off stale wheel_diameter item

Co-Authored-By: Claude Fable 5 <noreply@anthropic.com>

File: src/mentorpi_description/urdf/mecanum.xacro (robot description, xacro)
@@ -1,13 +1,13 @@
 <?xml version="1.0" ?>
 <!--
-  MentorPi mecanum body — geometry source-of-truth for sim and real robot.
-  IMPORTANT: 轮位置必须与 src/mentorpi_base/mentorpi_base/base_node.py:281-283
-  保持一致。当前值 (wheelbase=0.1368, track_width=0.1410) 是占位估计。
-  Part 1 标定完成后，需同时更新此处与 base_node.py。
-  TF root: base_footprint (REP-105 地面投影) → base_link (底盘几何中心)
-  Camera optical frames 与 Orbbec 驱动发布的 frame 名一致；真机加载 URDF 时，
-  让 Orbbec 驱动的 publish_tf=false 以避免 TF 冲突。
+  MentorPi mecanum geometry source of truth.
+  runtime_mode=false: complete offline/RViz model rooted at base_footprint.
+  runtime_mode=true: hardware TF model rooted at base_link; EKF owns
+  odom->base_link and the Orbbec driver owns camera-internal frames.
+  Wheel geometry is still an estimate and must stay synchronized with
+  mentorpi_base/base_node.py after drivetrain calibration.
 -->
 <robot name="mentorpi_mecanum" xmlns:xacro="http://ros.org/wiki/xacro">
+  <xacro:arg name="runtime_mode" default="false"/>
   <!-- ===== 几何参数（与 base_node.py 同步） ===== -->
   <xacro:property name="wheelbase"     value="0.1368"/>
@@ -23,10 +23,12 @@
   <material name="white"><color rgba="1 1 1 1"/></material>
   <!-- ===== Root: base_footprint (REP-105) ===== -->
-  <link name="base_footprint"/>
-  <joint name="base_footprint_to_base_link" type="fixed">
-    <parent link="base_footprint"/>
-    <child link="base_link"/>
-    <origin xyz="0 0 ${base_z}" rpy="0 0 0"/>
-  </joint>
+  <xacro:unless value="$(arg runtime_mode)">
+    <link name="base_footprint"/>
+    <joint name="base_footprint_to_base_link" type="fixed">
+      <parent link="base_footprint"/>
+      <child link="base_link"/>
+      <origin xyz="0 0 ${base_z}" rpy="0 0 0"/>
+    </joint>
+  </xacro:unless>
   <link name="base_link">
     <inertial>
@@ -76,13 +78,13 @@
   <xacro:mecanum_wheel prefix="lb" x="-${x_off}" y=" ${y_off}" mesh="wheel_lb_Link.STL"/>
   <xacro:mecanum_wheel prefix="rb" x="-${x_off}" y="-${y_off}" mesh="wheel_rb_Link.STL"/>
-  <!-- ===== IMU (Part 2 标定将更新 origin) ===== -->
+  <!-- ===== IMU (runtime estimate; Part 2 calibration pending) ===== -->
   <link name="imu_link"/>
   <joint name="imu_joint" type="fixed">
     <parent link="base_link"/>
     <child link="imu_link"/>
-    <!-- xyz 占位 (0,0,0)；rpy 来自 vendor mecanum.xacro。Part 2 完成后更新 -->
-    <origin xyz="0 0 0" rpy="0 0 ${-PI/2}"/>
+    <!-- Runtime estimate; refine position and axes in Part 2. -->
+    <origin xyz="0 0 0.05" rpy="0 0 0"/>
   </joint>
-  <!-- ===== Camera (Gemini 2L) — Part 3 标定将更新 origin ===== -->
+  <!-- ===== Camera (AprilTag hand-eye calibrated 2026-07-12) ===== -->
   <link name="camera_link">
     <inertial>
@@ -104,20 +106,22 @@
     <parent link="base_link"/>
     <child link="camera_link"/>
-    <!-- Vendor CAD 值；Part 3 AprilTag 标定后更新 -->
-    <origin xyz="0.061376 0 0.051154" rpy="0 0 0"/>
+    <!-- AprilTag hand-eye calibration, 2026-07-12; z is ruler-fixed. -->
+    <origin xyz="0.0846 0.0231 0.095" rpy="-0.0032 0.0149 -0.0422"/>
   </joint>
-  <!-- Optical frames: ROS REP-103 (z-forward, x-right, y-down). 与 Orbbec 驱动发的 frame 名一致 -->
-  <link name="camera_color_optical_frame"/>
-  <joint name="camera_color_optical_joint" type="fixed">
-    <parent link="camera_link"/>
-    <child link="camera_color_optical_frame"/>
-    <origin xyz="0 0 0" rpy="${-PI/2} 0 ${-PI/2}"/>
-  </joint>
-  <link name="camera_depth_optical_frame"/>
-  <joint name="camera_depth_optical_joint" type="fixed">
-    <parent link="camera_link"/>
-    <child link="camera_depth_optical_frame"/>
-    <origin xyz="0 0 0" rpy="${-PI/2} 0 ${-PI/2}"/>
-  </joint>
+  <!-- Offline preview only; Orbbec owns these frames on hardware. -->
+  <xacro:unless value="$(arg runtime_mode)">
+    <link name="camera_color_optical_frame"/>
+    <joint name="camera_color_optical_joint" type="fixed">
+      <parent link="camera_link"/>
+      <child link="camera_color_optical_frame"/>
+      <origin xyz="0 0 0" rpy="${-PI/2} 0 ${-PI/2}"/>
+    </joint>
+    <link name="camera_depth_optical_frame"/>
+    <joint name="camera_depth_optical_joint" type="fixed">
+      <parent link="camera_link"/>
+      <child link="camera_depth_optical_frame"/>
+      <origin xyz="0 0 0" rpy="${-PI/2} 0 ${-PI/2}"/>
+    </joint>
+  </xacro:unless>
   <!-- ===== Lidar (MS200) ===== -->
   <link name="laser_frame">
@@ -140,6 +144,6 @@
     <parent link="base_link"/>
     <child link="laser_frame"/>
-    <!-- Vendor CAD 值（mentorpi.launch.py 的 0.18 是错的占位估计，需同步更新） -->
-    <origin xyz="-0.012242 0 0.092501" rpy="0 0 0"/>
+    <!-- Current measured runtime value; x/y and RPY still need survey. -->
+    <origin xyz="0 0 0.18" rpy="0 0 0"/>
   </joint>
 </robot>

Commit message: calib: survey values + wheel_diameter sync + handoff doc
- mecanum.xacro: laser_joint x=-0.014 (lidar 1.4cm behind base center,
  y centered), imu_joint x=-0.054 (STM32 board 5.4cm behind; translation
  is cosmetic, only RPY axis alignment matters for gyro/gravity fusion),
  wheel_diameter 0.065 -> 0.0636 (was stale vs base_node Step 1.1 calib).
- TODO: flag camera extrinsic re-calibration after screw was re-tightened
  2026-07-14 (pitch likely shifted; must precede any daytime rescan).
- docs/calibration_handoff.md: cold-start handoff for continuing the
  real-robot calibration (remaining: gyro-z sign, rotation calib, 3x3m
  acceptance; battery died mid-work).

Co-Authored-By: Claude Fable 5 <noreply@anthropic.com>

File: src/mentorpi_description/urdf/mecanum.xacro (robot description, xacro)
@@ -13,5 +13,5 @@
   <xacro:property name="wheelbase"     value="0.1368"/>
   <xacro:property name="track_width"   value="0.1410"/>
-  <xacro:property name="wheel_diameter" value="0.065"/>
+  <xacro:property name="wheel_diameter" value="0.0636"/>  <!-- Step 1.1 calibrated 2026-07-05, synced with base_node.py -->
   <xacro:property name="wheel_radius"  value="${wheel_diameter/2}"/>
   <xacro:property name="x_off"         value="${wheelbase/2}"/>     <!-- 0.0684 -->
@@ -83,6 +83,10 @@
     <parent link="base_link"/>
     <child link="imu_link"/>
-    <!-- Runtime estimate; refine position and axes in Part 2. -->
-    <origin xyz="0 0 0.05" rpy="0 0 0"/>
+    <!-- STM32 board center ruler-measured 5.4cm behind base center, laterally
+         symmetric; z est. Translation is cosmetic: EKF fuses only gyro vyaw
+         and Madgwick only the gravity vector, both position-independent. Only
+         RPY axis alignment matters; static read (az≈+9.8, ax/ay small)
+         confirms z-up, no axis flip. Refine RPY in Part 2 if board is skewed. -->
+    <origin xyz="-0.054 0 0.05" rpy="0 0 0"/>
   </joint>
   <!-- ===== Camera (AprilTag hand-eye calibrated 2026-07-12) ===== -->
@@ -144,6 +148,7 @@
     <parent link="base_link"/>
     <child link="laser_frame"/>
-    <!-- Current measured runtime value; x/y and RPY still need survey. -->
-    <origin xyz="0 0 0.18" rpy="0 0 0"/>
+    <!-- x: ruler-measured 1.4cm behind base center; y: laterally centered;
+         z: measured. RPY (mounting yaw) still to be refined via wall line-fit. -->
+    <origin xyz="-0.014 0 0.18" rpy="0 0 0"/>
   </joint>
 </robot>

Commit message: calib: wall-rotation results — effective wheelbase/track + gyro_scale_z
Step 1.2: k_geom=1.117 (CCW 1.1049 / CW 1.1286, wall line-fit ground
truth, 2 turns each). wheelbase/track_width 0.1368/0.1410 ->
0.1528/0.1575 effective (absorbs in-place rotation roller slip) in
base_node._mecanum + mecanum.xacro, kept in sync.

Step 2.4: k_gyro=1.0071 (both directions agree -> true scale error).
New base_node param gyro_scale_z=0.9930, applied after bias removal,
hot-updatable.

Step 2 sign check: gz peak +0.64 rad/s during CCW -> REP-103 OK.

calibrate_rotation.py: fix report() summing signed direction totals
(CCW/CW cancel to ~0 making k values garbage) -> sum abs; update
script geometry constants to new effective values.

Docs: TODO 1.2/2.1/2.4 checked, handoff + CLAUDE.md updated.

Co-Authored-By: Claude Fable 5 <noreply@anthropic.com>

File: src/mentorpi_description/urdf/mecanum.xacro (robot description, xacro)
@@ -11,6 +11,9 @@
   <xacro:arg name="runtime_mode" default="false"/>
   <!-- ===== 几何参数（与 base_node.py 同步） ===== -->
-  <xacro:property name="wheelbase"     value="0.1368"/>
-  <xacro:property name="track_width"   value="0.1410"/>
+  <!-- 有效轴距 (Step 1.2 对墙旋转标定 2026-07-16, k_geom=1.117, 与
+       base_node.py _mecanum 同步; 物理尺量 0.1368/0.1410, 差值为麦轮
+       原地旋转打滑 → 轮子视觉位置比实物略外扩 ~8mm, 属已知取舍) -->
+  <xacro:property name="wheelbase"     value="0.1528"/>
+  <xacro:property name="track_width"   value="0.1575"/>
   <xacro:property name="wheel_diameter" value="0.0636"/>  <!-- Step 1.1 calibrated 2026-07-05, synced with base_node.py -->
   <xacro:property name="wheel_radius"  value="${wheel_diameter/2}"/>

Commit message: calib: camera extrinsic re-solved after screw re-tightening (2026-07-17)
AprilTag hand-eye, 8 poses (4 arc + 4 line), residual RMS 9.7mm.
pitch moved +0.85deg -> -7.46deg vs the 2026-07-12 solve — confirms the
loosened-screw invalidation. x/y/yaw shifted accordingly (z ruler-fixed).

Co-Authored-By: Claude Fable 5 <noreply@anthropic.com>

File: src/mentorpi_description/urdf/mecanum.xacro (robot description, xacro)
@@ -113,6 +113,6 @@
     <parent link="base_link"/>
     <child link="camera_link"/>
-    <!-- AprilTag hand-eye calibration, 2026-07-12; z is ruler-fixed. -->
-    <origin xyz="0.0846 0.0231 0.095" rpy="-0.0032 0.0149 -0.0422"/>
+    <!-- AprilTag hand-eye calibration, 2026-07-17; z is ruler-fixed. -->
+    <origin xyz="0.1114 0.0305 0.0950" rpy="-0.0164 -0.1302 0.0147"/>
   </joint>
   <!-- Offline preview only; Orbbec owns these frames on hardware. -->

Commit message: vendor: SO-101 integration draft (Codex snapshot, as-received)
Codex's first-pass MentorPi × SO-101 integration: so101.xacro conversion
pipeline (upstream SO-ARM100 fda892c), 13 arm meshes, 4 parametric printable
parts (adapter plate / anker tray / lidar riser / hub carrier) with
STEP+STL+snapshots, with_so101 xacro branch, clearance check script, and the
implementation report (docs/mentorpi_so101_integration_report.md).

Committed as-received for provenance. Known issues from review (to be
addressed in follow-up commits): no runtime with_so101 plumbing, unconditional
so101.xacro include, riser invalidates maps/guard coverage, arm faces rear,
PD power ceiling. Redesign follows: arm-forward + lidar-stays-masked + 2S
direct power.

Co-Authored-By: Claude Fable 5 <noreply@anthropic.com>

File: src/mentorpi_description/urdf/mecanum.xacro (robot description, xacro)
@@ -10,4 +10,6 @@
 <robot name="mentorpi_mecanum" xmlns:xacro="http://ros.org/wiki/xacro">
   <xacro:arg name="runtime_mode" default="false"/>
+  <xacro:arg name="with_so101" default="false"/>
+  <xacro:include filename="$(find mentorpi_description)/urdf/so101.xacro"/>
   <!-- ===== 几何参数（与 base_node.py 同步） ===== -->
   <!-- 有效轴距 (Step 1.2 对墙旋转标定 2026-07-16, k_geom=1.117, 与
@@ -148,10 +150,117 @@
     </collision>
   </link>
-  <joint name="laser_joint" type="fixed">
-    <parent link="base_link"/>
-    <child link="laser_frame"/>
-    <!-- x: ruler-measured 1.4cm behind base center; y: laterally centered;
-         z: measured. RPY (mounting yaw) still to be refined via wall line-fit. -->
-    <origin xyz="-0.014 0 0.18" rpy="0 0 0"/>
-  </joint>
+  <xacro:unless value="$(arg with_so101)">
+    <joint name="laser_joint" type="fixed">
+      <parent link="base_link"/>
+      <child link="laser_frame"/>
+      <!-- x: ruler-measured 1.4cm behind base center; y: laterally centered;
+           z: measured. RPY (mounting yaw) still to be refined via wall line-fit. -->
+      <origin xyz="-0.014 0 0.18" rpy="0 0 0"/>
+    </joint>
+  </xacro:unless>
+  <xacro:if value="$(arg with_so101)">
+    <joint name="laser_joint" type="fixed">
+      <parent link="base_link"/>
+      <child link="laser_frame"/>
+      <!-- 170 mm printable riser clears the official new-calibration zero pose. -->
+      <origin xyz="-0.014 0 0.35" rpy="0 0 0"/>
+    </joint>
+    <xacro:so101_module
+      parent="base_link"
+      mount_xyz="-0.0409 0 0.0655"
+      mount_rpy="0 0 ${PI}"/>
+    <!-- Printed adapter: measured rear spare-hole center + top-plate height. -->
+    <link name="so101_adapter_link">
+      <inertial>
+        <origin xyz="0 0 0.004" rpy="0 0 0"/>
+        <mass value="0.18"/>
+        <inertia ixx="0.000112" ixy="0" ixz="0"
+                 iyy="0.000209" iyz="0" izz="0.000221"/>
+      </inertial>
+      <visual>
+        <geometry>
+          <mesh filename="package://mentorpi_description/meshes/accessories/arm_adapter_plate.stl"
+                scale="0.001 0.001 0.001"/>
+        </geometry>
+        <material name="adapter_orange"><color rgba="0.95 0.35 0.08 1"/></material>
+      </visual>
+      <collision>
+        <origin xyz="0 0 0.004" rpy="0 0 0"/>
+        <geometry><box size="0.118 0.086 0.008"/></geometry>
+      </collision>
+    </link>
+    <joint name="so101_adapter_joint" type="fixed">
+      <parent link="base_link"/>
+      <child link="so101_adapter_link"/>
+      <origin xyz="-0.0409 0 0.0575" rpy="0 0 0"/>
+    </joint>
+    <!-- Low front counterweight tray and A1335 envelope; both stay below camera. -->
+    <link name="anker_tray_link">
+      <inertial>
+        <origin xyz="-0.004 0 0.020" rpy="0 0 0"/>
+        <mass value="0.12"/>
+        <inertia ixx="0.00023" ixy="0" ixz="0"
+                 iyy="0.00005" iyz="0" izz="0.00022"/>
+      </inertial>
+      <visual>
+        <geometry>
+          <mesh filename="package://mentorpi_description/meshes/accessories/anker_prime_front_tray.stl"
+                scale="0.001 0.001 0.001"/>
+        </geometry>
+        <material name="tray_blue"><color rgba="0.10 0.35 0.80 1"/></material>
+      </visual>
+      <collision>
+        <origin xyz="-0.004 0 0.029" rpy="0 0 0"/>
+        <geometry><box size="0.05013 0.142 0.058"/></geometry>
+      </collision>
+    </link>
+    <joint name="anker_tray_joint" type="fixed">
+      <parent link="base_link"/>
+      <child link="anker_tray_link"/>
+      <origin xyz="0.130 0 -0.003" rpy="0 0 0"/>
+    </joint>
+    <link name="anker_prime_link">
+      <inertial>
+        <origin xyz="0 0 0" rpy="0 0 0"/>
+        <mass value="0.36"/>
+        <inertia ixx="0.000633" ixy="0" ixz="0"
+                 iyy="0.000127" iyz="0" izz="0.000578"/>
+      </inertial>
+      <visual>
+        <geometry><box size="0.03453 0.1344 0.055"/></geometry>
+        <material name="anker_gray"><color rgba="0.16 0.17 0.19 1"/></material>
+      </visual>
+      <collision><geometry><box size="0.03453 0.1344 0.055"/></geometry></collision>
+    </link>
+    <joint name="anker_prime_joint" type="fixed">
+      <parent link="base_link"/>
+      <child link="anker_prime_link"/>
+      <origin xyz="0.130 0 0.0305" rpy="0 0 0"/>
+    </joint>
+    <!-- Riser bottom sits at the former laser mounting plane; top is z=0.350 m. -->
+    <link name="lidar_riser_link">
+      <inertial>
+        <origin xyz="0 0 0.0875" rpy="0 0 0"/>
+        <mass value="0.10"/>
+        <inertia ixx="0.00020" ixy="0" ixz="0"
+                 iyy="0.00020" iyz="0" izz="0.00005"/>
+      </inertial>
+      <visual>
+        <geometry>
+          <mesh filename="package://mentorpi_description/meshes/accessories/lidar_riser.stl"
+                scale="0.001 0.001 0.001"/>
+        </geometry>
+        <material name="riser_orange"><color rgba="0.95 0.35 0.08 1"/></material>
+      </visual>
+      <collision>
+        <origin xyz="-0.022 0 0.0875" rpy="0 0 0"/>
+        <geometry><box size="0.012 0.050 0.175"/></geometry>
+      </collision>
+    </link>
+    <joint name="lidar_riser_joint" type="fixed">
+      <parent link="base_link"/>
+      <child link="lidar_riser_link"/>
+      <origin xyz="-0.014 0 0.175" rpy="0 0 0"/>
+    </joint>
+  </xacro:if>
 </robot>
