Commit message: urdf: SO-101 layout v2 — arm forward, lidar stays, visual fixes
Replaces the Codex rear-facing + 170mm-riser layout:
- so101 mount yaw 0 (forward): Gemini 2L becomes the VLA context camera,
  gripper enters frame when reaching. Mount x=-0.155 chosen by real-mesh
  pan-sweep (±110°): worst clearance 23.1mm to lidar head, 11.4mm to the
  assumed tower posts (zero pose: 66.9/25.2/11.5mm).
- laser_joint stays at z=0.18 in both configs — existing 2D/3D maps remain
  valid; the stowed arm's rear sector is handled by a laser_filters mask
  (base.launch.py), not by raising the lidar.
- so101.xacro include moved inside the with_so101 if-block (xacro evaluates
  lazily) — tracked files no longer hard-depend on it when the arm is off.
- camera visual: cam_Link.STL is body-centered; camera_link is the
  calibrated optical center (lens ~3cm off-center, front face, mid-height).
  Cosmetic mesh offset added so the body renders where it physically is;
  calibrated camera_joint untouched (ground-plane verified).
- lidar tower posts drawn as cosmetic visuals (base_link.STL omits the
  tower — the lidar head used to float 9cm above the deck).
- riser / anker tray / A1335 links removed; deck is a placeholder box until
  the P2 CAD part lands.

Co-Authored-By: Claude Fable 5 <noreply@anthropic.com>

File: src/mentorpi_description/urdf/mecanum.xacro (robot description, xacro)
@@ -10,6 +10,7 @@
 <robot name="mentorpi_mecanum" xmlns:xacro="http://ros.org/wiki/xacro">
   <xacro:arg name="runtime_mode" default="false"/>
+  <!-- with_so101: SO-101 机械臂车载布局。include 放在 if 块内(xacro 惰性求值),
+       未启用时不依赖 so101.xacro 存在。 -->
   <xacro:arg name="with_so101" default="false"/>
-  <xacro:include filename="$(find mentorpi_description)/urdf/so101.xacro"/>
   <!-- ===== 几何参数（与 base_node.py 同步） ===== -->
   <!-- 有效轴距 (Step 1.2 对墙旋转标定 2026-07-16, k_geom=1.117, 与
@@ -102,11 +103,15 @@
       <inertia ixx="1.44E-05" ixy="0" ixz="0" iyy="1.66E-06" iyz="0" izz="1.46E-05"/>
     </inertial>
-    <visual>
-      <origin rpy="0 0 0" xyz="0 0 0"/>
+    <!-- 视觉修正(纯外观): cam_Link.STL 以机身顶面中心为原点建模,而
+         camera_link 是标定出的光学中心——彩色镜头偏离机身中心 ~3cm(y),
+         位于前脸(x)、中高(z)。不加偏移时机身网格会整体跟着光学系平移,
+         看起来"装歪"。标定值本身经地面点云验证,勿动 camera_joint。 -->
+    <visual>
+      <origin rpy="0 0 0" xyz="-0.0137 -0.0305 0.013"/>
       <geometry><mesh filename="package://mentorpi_description/meshes/mecanum/cam_Link.STL"/></geometry>
       <material name="black"/>
     </visual>
     <collision>
-      <origin rpy="0 0 0" xyz="0 0 0"/>
+      <origin rpy="0 0 0" xyz="-0.0137 -0.0305 0.013"/>
       <geometry><mesh filename="package://mentorpi_description/meshes/mecanum/cam_Link.STL"/></geometry>
     </collision>
@@ -150,116 +155,71 @@
     </collision>
   </link>
-  <xacro:unless value="$(arg with_so101)">
-    <joint name="laser_joint" type="fixed">
-      <parent link="base_link"/>
-      <child link="laser_frame"/>
-      <!-- x: ruler-measured 1.4cm behind base center; y: laterally centered;
-           z: measured. RPY (mounting yaw) still to be refined via wall line-fit. -->
-      <origin xyz="-0.014 0 0.18" rpy="0 0 0"/>
-    </joint>
-  </xacro:unless>
+  <joint name="laser_joint" type="fixed">
+    <parent link="base_link"/>
+    <child link="laser_frame"/>
+    <!-- x: ruler-measured 1.4cm behind base center; y: laterally centered;
+         z: measured. RPY (mounting yaw) still to be refined via wall line-fit.
+         装臂(with_so101)不改变雷达高度——臂占据的后向扇区由 laser_filters
+         角度掩膜滤除(见 base.launch.py),现有 2D/3D 地图资产保持有效。 -->
+    <origin xyz="-0.014 0 0.18" rpy="0 0 0"/>
+  </joint>
+  <!-- 雷达塔架(纯外观): base_link.STL 不含塔架,雷达头会悬浮在顶板上方
+       ~9cm。4 根立柱位置 = Codex 网格分析推测的后部 Ø4.3 孔位,与实物
+       待卡尺核对(P0);画出来只为骨架可读,不参与任何 TF/碰撞。 -->
+  <xacro:macro name="lidar_post" params="x y">
+    <visual>
+      <origin xyz="${x} ${y} 0.10125" rpy="0 0 0"/>
+      <geometry><cylinder radius="0.004" length="0.0875"/></geometry>
+      <material name="black"/>
+    </visual>
+  </xacro:macro>
+  <link name="lidar_mount_visual_link">
+    <xacro:lidar_post x="-0.0509" y=" 0.0244"/>
+    <xacro:lidar_post x="-0.0509" y="-0.0244"/>
+    <xacro:lidar_post x="-0.0309" y=" 0.0244"/>
+    <xacro:lidar_post x="-0.0309" y="-0.0244"/>
+  </link>
+  <joint name="lidar_mount_visual_joint" type="fixed">
+    <parent link="base_link"/>
+    <child link="lidar_mount_visual_link"/>
+    <origin xyz="0 0 0" rpy="0 0 0"/>
+  </joint>
+  <!-- ===== SO-101 机械臂(可选, with_so101:=true) =====
+       布局 v2(2026-07-18, 取代 Codex 朝后+riser 方案):
+       - 臂朝前(yaw 0): Gemini 2L 天然成为 VLA context 相机,前伸时夹爪入画
+       - 雷达不动: 保住已建地图与低障碍探测;臂收拢姿态占据的后向扇区
+         用激光角度掩膜滤除;抓取作业时停车(motion primitive 安全模型)
+       - 臂基座后移至 x=-0.155: 真网格 pan 全程(±110°)扫掠最差裕量
+         头部 23.1mm / 推测立柱 11.4mm(v2_pan.py, 2026-07-18);甲板从
+         共用锚点向后悬伸 ~92mm,SO-101 越过雷达头上方前伸作业
+       - 甲板 deck 为占位 box,P2 CAD 出真实网格后替换 -->
   <xacro:if value="$(arg with_so101)">
-    <joint name="laser_joint" type="fixed">
-      <parent link="base_link"/>
-      <child link="laser_frame"/>
-      <!-- 170 mm printable riser clears the official new-calibration zero pose. -->
-      <origin xyz="-0.014 0 0.35" rpy="0 0 0"/>
-    </joint>
+    <xacro:include filename="$(find mentorpi_description)/urdf/so101.xacro"/>
     <xacro:so101_module
       parent="base_link"
-      mount_xyz="-0.0409 0 0.0655"
-      mount_rpy="0 0 ${PI}"/>
-    <!-- Printed adapter: measured rear spare-hole center + top-plate height. -->
-    <link name="so101_adapter_link">
+      mount_xyz="-0.155 0 0.0655"
+      mount_rpy="0 0 0"/>
+    <!-- 悬伸甲板占位: x -0.195..-0.015, y ±0.048, 顶面 z=0.0655 -->
+    <link name="so101_deck_link">
       <inertial>
-        <origin xyz="0 0 0.004" rpy="0 0 0"/>
-        <mass value="0.18"/>
-        <inertia ixx="0.000112" ixy="0" ixz="0"
-                 iyy="0.000209" iyz="0" izz="0.000221"/>
+        <origin xyz="-0.105 0 -0.004" rpy="0 0 0"/>
+        <mass value="0.19"/>
+        <inertia ixx="0.000147" ixy="0" ixz="0"
+                 iyy="0.000515" iyz="0" izz="0.000659"/>
       </inertial>
       <visual>
-        <geometry>
-          <mesh filename="package://mentorpi_description/meshes/accessories/arm_adapter_plate.stl"
-                scale="0.001 0.001 0.001"/>
-        </geometry>
-        <material name="adapter_orange"><color rgba="0.95 0.35 0.08 1"/></material>
+        <origin xyz="-0.105 0 -0.004" rpy="0 0 0"/>
+        <geometry><box size="0.180 0.096 0.008"/></geometry>
+        <material name="deck_orange"><color rgba="0.95 0.35 0.08 1"/></material>
       </visual>
       <collision>
-        <origin xyz="0 0 0.004" rpy="0 0 0"/>
-        <geometry><box size="0.118 0.086 0.008"/></geometry>
+        <origin xyz="-0.105 0 -0.004" rpy="0 0 0"/>
+        <geometry><box size="0.180 0.096 0.008"/></geometry>
       </collision>
     </link>
-    <joint name="so101_adapter_joint" type="fixed">
+    <joint name="so101_deck_joint" type="fixed">
       <parent link="base_link"/>
-      <child link="so101_adapter_link"/>
-      <origin xyz="-0.0409 0 0.0575" rpy="0 0 0"/>
-    </joint>
-    <!-- Low front counterweight tray and A1335 envelope; both stay below camera. -->
-    <link name="anker_tray_link">
-      <inertial>
-        <origin xyz="-0.004 0 0.020" rpy="0 0 0"/>
-        <mass value="0.12"/>
-        <inertia ixx="0.00023" ixy="0" ixz="0"
-                 iyy="0.00005" iyz="0" izz="0.00022"/>
-      </inertial>
-      <visual>
-        <geometry>
-          <mesh filename="package://mentorpi_description/meshes/accessories/anker_prime_front_tray.stl"
-                scale="0.001 0.001 0.001"/>
-        </geometry>
-        <material name="tray_blue"><color rgba="0.10 0.35 0.80 1"/></material>
-      </visual>
-      <collision>
-        <origin xyz="-0.004 0 0.029" rpy="0 0 0"/>
-        <geometry><box size="0.05013 0.142 0.058"/></geometry>
-      </collision>
-    </link>
-    <joint name="anker_tray_joint" type="fixed">
-      <parent link="base_link"/>
-      <child link="anker_tray_link"/>
-      <origin xyz="0.130 0 -0.003" rpy="0 0 0"/>
-    </joint>
-    <link name="anker_prime_link">
-      <inertial>
-        <origin xyz="0 0 0" rpy="0 0 0"/>
-        <mass value="0.36"/>
-        <inertia ixx="0.000633" ixy="0" ixz="0"
-                 iyy="0.000127" iyz="0" izz="0.000578"/>
-      </inertial>
-      <visual>
-        <geometry><box size="0.03453 0.1344 0.055"/></geometry>
-        <material name="anker_gray"><color rgba="0.16 0.17 0.19 1"/></material>
-      </visual>
-      <collision><geometry><box size="0.03453 0.1344 0.055"/></geometry></collision>
-    </link>
-    <joint name="anker_prime_joint" type="fixed">
-      <parent link="base_link"/>
-      <child link="anker_prime_link"/>
-      <origin xyz="0.130 0 0.0305" rpy="0 0 0"/>
-    </joint>
-    <!-- Riser bottom sits at the former laser mounting plane; top is z=0.350 m. -->
-    <link name="lidar_riser_link">
-      <inertial>
-        <origin xyz="0 0 0.0875" rpy="0 0 0"/>
-        <mass value="0.10"/>
-        <inertia ixx="0.00020" ixy="0" ixz="0"
-                 iyy="0.00020" iyz="0" izz="0.00005"/>
-      </inertial>
-      <visual>
-        <geometry>
-          <mesh filename="package://mentorpi_description/meshes/accessories/lidar_riser.stl"
-                scale="0.001 0.001 0.001"/>
-        </geometry>
-        <material name="riser_orange"><color rgba="0.95 0.35 0.08 1"/></material>
-      </visual>
-      <collision>
-        <origin xyz="-0.022 0 0.0875" rpy="0 0 0"/>
-        <geometry><box size="0.012 0.050 0.175"/></geometry>
-      </collision>
-    </link>
-    <joint name="lidar_riser_joint" type="fixed">
-      <parent link="base_link"/>
-      <child link="lidar_riser_link"/>
-      <origin xyz="-0.014 0 0.175" rpy="0 0 0"/>
+      <child link="so101_deck_link"/>
+      <origin xyz="0 0 0.0655" rpy="0 0 0"/>
     </joint>
   </xacro:if>

Commit message: mech: layout v2 CAD — cantilever deck + 2S battery tray
so101_deck_plate: 180x96x8 rear cantilever deck, shim-mode anchors on the
four Codex-inferred chassis holes (M4 through + counterbore, lidar tower
standoffs re-bolt through), SO-101 M4 grid + strap slots, twin 15mm
underside ribs + rear web on the 92mm cantilever. battery_tray_2s: front-
hung tray for the arm's dedicated 2S pack (provisional 105x33x24 envelope),
proper L-hooks (throat 6mm + drop-tab + M4 clamp — v1's hook lip could only
touch the edge arris), doubles as front counterweight.

URDF: deck placeholder box replaced with the real mesh; battery tray + pack
links added (with_so101 only). mentorpi_so101.urdf regenerated.

Analysis preserved as mechanical/measurements/check_so101_clearances.py
(real-mesh zero-pose + shoulder_pan sweep vs lidar head and assumed posts;
v2 numbers reproduced: 66.9/25.2/11.5mm zero pose, 23.1/11.4mm worst
sweep). check_urdf_clearances.py updated for v2 link names. mechanical
README + design ledger rewritten for v2 with the P0 caliper-audit checklist;
CLAUDE.md gains the integration section.

All parts remain parametric — update CHASSIS_HOLES / POSTS / PACK_* /
HOOK_THROAT after physical measurement and re-run the generators.

Co-Authored-By: Claude Fable 5 <noreply@anthropic.com>

File: src/mentorpi_description/urdf/mecanum.xacro (robot description, xacro)
@@ -200,5 +200,6 @@
       mount_xyz="-0.155 0 0.0655"
       mount_rpy="0 0 0"/>
-    <!-- 悬伸甲板占位: x -0.195..-0.015, y ±0.048, 顶面 z=0.0655 -->
+    <!-- 悬伸甲板 (mechanical/printable/so101_deck_plate.py):
+         x -0.195..-0.015, y ±0.048, 顶面 z=0.0655, 底面纵肋 15 深 -->
     <link name="so101_deck_link">
       <inertial>
@@ -209,6 +210,9 @@
       </inertial>
       <visual>
-        <origin xyz="-0.105 0 -0.004" rpy="0 0 0"/>
-        <geometry><box size="0.180 0.096 0.008"/></geometry>
+        <origin xyz="-0.105 0 -0.008" rpy="0 0 0"/>
+        <geometry>
+          <mesh filename="package://mentorpi_description/meshes/accessories/so101_deck_plate.stl"
+                scale="0.001 0.001 0.001"/>
+        </geometry>
         <material name="deck_orange"><color rgba="0.95 0.35 0.08 1"/></material>
       </visual>
@@ -223,4 +227,50 @@
       <origin xyz="0 0 0.0655" rpy="0 0 0"/>
     </joint>
+    <!-- 臂供电 2S 锂电: 前挂托架 (mechanical/printable/battery_tray_2s.py),
+         兼作前配重抗后倾。包络暂按 2S2200 (105x33x24) —— 购得实物后改
+         PACK_* 重出。托架背面贴底盘前脸 (x=0.109), 挂唇压顶缘。 -->
+    <link name="battery_tray_link">
+      <inertial>
+        <origin xyz="0 0 0.010" rpy="0 0 0"/>
+        <mass value="0.06"/>
+        <inertia ixx="0.00008" ixy="0" ixz="0"
+                 iyy="0.00002" iyz="0" izz="0.00009"/>
+      </inertial>
+      <visual>
+        <origin xyz="0 0 0" rpy="0 0 0"/>
+        <geometry>
+          <mesh filename="package://mentorpi_description/meshes/accessories/battery_tray_2s.stl"
+                scale="0.001 0.001 0.001"/>
+        </geometry>
+        <material name="tray_blue"><color rgba="0.10 0.35 0.80 1"/></material>
+      </visual>
+      <collision>
+        <origin xyz="0 0 0.0155" rpy="0 0 0"/>
+        <geometry><box size="0.0406 0.1126 0.031"/></geometry>
+      </collision>
+    </link>
+    <joint name="battery_tray_joint" type="fixed">
+      <parent link="base_link"/>
+      <child link="battery_tray_link"/>
+      <origin xyz="0.1293 0 0.0305" rpy="0 0 0"/>
+    </joint>
+    <link name="battery_2s_link">
+      <inertial>
+        <origin xyz="0 0 0" rpy="0 0 0"/>
+        <mass value="0.18"/>
+        <inertia ixx="0.000174" ixy="0" ixz="0"
+                 iyy="0.0000250" iyz="0" izz="0.000182"/>
+      </inertial>
+      <visual>
+        <geometry><box size="0.033 0.105 0.024"/></geometry>
+        <material name="lipo_gray"><color rgba="0.25 0.26 0.30 1"/></material>
+      </visual>
+      <collision><geometry><box size="0.033 0.105 0.024"/></geometry></collision>
+    </link>
+    <joint name="battery_2s_joint" type="fixed">
+      <parent link="battery_tray_link"/>
+      <child link="battery_2s_link"/>
+      <origin xyz="0 0 0.015" rpy="0 0 0"/>
+    </joint>
   </xacro:if>
 </robot>

File: src/mentorpi_description/urdf/mentorpi_so101.urdf (robot description, URDF)
Before this commit: robot mentorpi, 23 links, 22 joints
Links:
- removed link anker_prime_link
- removed link anker_tray_link
- removed link lidar_riser_link
- removed link so101_adapter_link
- added link battery_2s_link, mass 0.18; collision box size=0.033 0.105 0.024; visual box size=0.033 0.105 0.024
- added link battery_tray_link, mass 0.06; collision box size=0.0406 0.1126 0.031; visual mesh filename=package://mentorpi_description/meshes/accessories/battery_t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 scale=0.001 0.001 0.001
- added link lidar_mount_visual_link; visual cylinder length=0.0875 radius=0.004; visual cylinder length=0.0875 radius=0.004
- added link so101_deck_link, mass 0.19; collision box size=0.180 0.096 0.008; visual mesh filename=package://mentorpi_description/meshes/accessories/so101_dec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 scale=0.001 0.001 0.001
Joints:
- removed joint anker_prime_joint
- removed joint anker_tray_joint
- removed joint lidar_riser_joint
- removed joint so101_adapter_joint
- added joint battery_2s_joint: type fixed, parent battery_tray_link, child battery_2s_link, origin xyz=0 0 0.015 rpy=0 0 0
- added joint battery_tray_joint: type fixed, parent base_link, child battery_tray_link, origin xyz=0.1293 0 0.0305 rpy=0 0 0
- added joint lidar_mount_visual_joint: type fixed, parent base_link, child lidar_mount_visual_link, origin xyz=0 0 0 rpy=0 0 0
- added joint so101_deck_joint: type fixed, parent base_link, child so101_deck_link, origin xyz=0 0 0.0655 rpy=0 0 0
- joint laser_joint: origin xyz=-0.014 0 0.35 rpy=0 0 0 -> xyz=-0.014 0 0.18 rpy=0 0 0
- joint so101_mount_joint: origin xyz=-0.0409 0 0.0655 rpy=0 0 3.141592653589793 -> xyz=-0.155 0 0.0655 rpy=0 0 0

Commit message: viewer: strip collisions from preview URDF; add gimbal base visual
Collision blocks duplicated ~60MB of STL parsing in the browser (mecanum
wheel meshes are 9.8MB each) — preview variant is visual-only now. Also
draw the camera gimbal base (top plate to camera body, absent from vendor
meshes, same story as the lidar tower).

Co-Authored-By: Claude Fable 5 <noreply@anthropic.com>

File: src/mentorpi_description/urdf/mecanum.xacro (robot description, xacro)
@@ -179,4 +179,11 @@
     <xacro:lidar_post x="-0.0309" y=" 0.0244"/>
     <xacro:lidar_post x="-0.0309" y="-0.0244"/>
+    <!-- 相机云台底座(纯外观): 顶板(0.0575)到相机机身底(~0.077)之间的
+         2-DOF 云台舵机组,同样不在任何厂商网格里。 -->
+    <visual>
+      <origin xyz="0.093 0 0.0675" rpy="0 0 0"/>
+      <geometry><box size="0.030 0.040 0.020"/></geometry>
+      <material name="black"/>
+    </visual>
   </link>
   <joint name="lidar_mount_visual_joint" type="fixed">

File: src/mentorpi_description/urdf/mentorpi_so101.urdf (robot description, URDF)
Before this commit: robot mentorpi, 23 links, 22 joints
Links:
- link lidar_mount_visual_link: geometry visual box size=0.030 0.040 0.020; visual cylinder length=0.0875 radius=0.004

File: src/mentorpi_description/urdf/mentorpi_so101.viewer.urdf (robot description, URDF)
Before this commit: robot mentorpi, 23 links, 22 joints
Links:
- link base_link: geometry visual mesh filename=../meshes/mecanum/base_link.STL
- link battery_2s_link: geometry visual box size=0.033 0.105 0.024
- link battery_tray_link: geometry visual mesh filename=../meshes/accessories/battery_tray_2s.stl scale=0.001 0.001 0.001
- link camera_link: geometry visual mesh filename=../meshes/mecanum/cam_Link.STL
- link laser_frame: geometry visual mesh filename=../meshes/mecanum/lidar_Link.STL
- link lidar_mount_visual_link: geometry visual box size=0.030 0.040 0.020; visual cylinder length=0.0875 radius=0.004
- link so101_base_link: geometry visual mesh filename=../meshes/so101/base_motor_holder_so101_v1.stl; visual mesh filename=../meshes/so101/base_so101_v2.stl
- link so101_deck_link: geometry visual mesh filename=../meshes/accessories/so101_deck_plate.stl scale=0.001 0.001 0.001
- link so101_gripper_link: geometry visual mesh filename=../meshes/so101/sts3215_03a_v1.stl; visual mesh filename=../meshes/so101/wrist_roll_follower_so101_v1.stl
- link so101_lower_arm_link: geometry visual mesh filename=../meshes/so101/motor_holder_so101_wrist_v1.stl; visual mesh filename=../meshes/so101/sts3215_03a_v1.stl
- link so101_moving_jaw_so101_v1_link: geometry visual mesh filename=../meshes/so101/moving_jaw_so101_v1.stl
- link so101_shoulder_link: geometry visual mesh filename=../meshes/so101/motor_holder_so101_base_v1.stl; visual mesh filename=../meshes/so101/rotation_pitch_so101_v1.stl
- link so101_upper_arm_link: geometry visual mesh filename=../meshes/so101/sts3215_03a_v1.stl; visual mesh filename=../meshes/so101/upper_arm_so101_v1.stl
- link so101_wrist_link: geometry visual mesh filename=../meshes/so101/sts3215_03a_no_horn_v1.stl; visual mesh filename=../meshes/so101/wrist_roll_pitch_so101_v2.stl
- link wheel_lb_Link: geometry visual mesh filename=../meshes/mecanum/wheel_lb_Link.STL
- link wheel_lf_Link: geometry visual mesh filename=../meshes/mecanum/wheel_lf_Link.STL
- link wheel_rb_Link: geometry visual mesh filename=../meshes/mecanum/wheel_rb_Link.STL
- link wheel_rf_Link: geometry visual mesh filename=../meshes/mecanum/wheel_rf_Link.STL

Commit message: urdf: fix two real floaters — gimbal tower + battery hang line
User's GLB screenshot showed genuine gaps (not a loader bug this time).
Mesh slicing of base_link.STL proved the chassis nose is STEPPED: the
57.5mm top plate ends at x=+17mm, a mid deck at z=25.3mm runs to x=+80mm,
and only a low bumper reaches the true front — the vertical front face my
battery tray hooks targeted does not exist.

- battery tray re-hung on the mid-deck front edge (back face x=0.080, lip
  on z=0.0253); tray CAD unchanged (parametric), joint + docstring updated.
  Bonus: pack top drops from z=0.108 to 0.0253 — camera clearance grows
  from 16mm to ~52mm.
- gimbal token box replaced with the full servo tower (z 0.0253..0.0772,
  52mm tall, absent from vendor meshes).

Offline orthographic re-render confirms all visuals connect.

Co-Authored-By: Claude Fable 5 <noreply@anthropic.com>

File: src/mentorpi_description/urdf/mecanum.xacro (robot description, xacro)
@@ -179,9 +179,11 @@
     <xacro:lidar_post x="-0.0309" y=" 0.0244"/>
     <xacro:lidar_post x="-0.0309" y="-0.0244"/>
-    <!-- 相机云台底座(纯外观): 顶板(0.0575)到相机机身底(~0.077)之间的
-         2-DOF 云台舵机组,同样不在任何厂商网格里。 -->
-    <visual>
-      <origin xyz="0.093 0 0.0675" rpy="0 0 0"/>
-      <geometry><box size="0.030 0.040 0.020"/></geometry>
+    <!-- 相机云台舵机塔(纯外观): 网格切片实测底盘鼻部是台阶状——顶板
+         (z=0.0575)只到 x≈+0.017,前方是 z≈0.0253 的中层甲板(到 x≈0.08)。
+         2-DOF 云台从中层甲板(0.0253)撑到相机机身底(0.0772),高 52mm,
+         不在任何厂商网格里。 -->
+    <visual>
+      <origin xyz="0.088 0 0.0513" rpy="0 0 0"/>
+      <geometry><box size="0.028 0.040 0.052"/></geometry>
       <material name="black"/>
     </visual>
@@ -236,5 +238,6 @@
     <!-- 臂供电 2S 锂电: 前挂托架 (mechanical/printable/battery_tray_2s.py),
          兼作前配重抗后倾。包络暂按 2S2200 (105x33x24) —— 购得实物后改
-         PACK_* 重出。托架背面贴底盘前脸 (x=0.109), 挂唇压顶缘。 -->
+         PACK_* 重出。挂线(网格切片实测,P0 卡尺复核): 底盘鼻部无垂直
+         前脸——托架背面贴中层甲板前缘 x=0.080, 挂唇压其顶面 z=0.0253。 -->
     <link name="battery_tray_link">
       <inertial>
@@ -260,5 +263,7 @@
       <parent link="base_link"/>
       <child link="battery_tray_link"/>
-      <origin xyz="0.1293 0 0.0305" rpy="0 0 0"/>
+      <!-- 背面 x = 0.080 - outer_x/2 + outer_x = 0.0203+0.080; 挂唇底
+           z = -0.0017 + 0.027 = 0.0253 (中层甲板顶面)。 -->
+      <origin xyz="0.1003 0 -0.0017" rpy="0 0 0"/>
     </joint>
     <link name="battery_2s_link">

File: src/mentorpi_description/urdf/mentorpi_so101.urdf (robot description, URDF)
Before this commit: robot mentorpi, 23 links, 22 joints
Links:
- link lidar_mount_visual_link: geometry visual box size=0.028 0.040 0.052; visual cylinder length=0.0875 radius=0.004
Joints:
- joint battery_tray_joint: origin xyz=0.1293 0 0.0305 rpy=0 0 0 -> xyz=0.1003 0 -0.0017 rpy=0 0 0

File: src/mentorpi_description/urdf/mentorpi_so101.viewer.urdf (robot description, URDF)
Before this commit: robot mentorpi, 23 links, 22 joints
Links:
- link lidar_mount_visual_link: geometry visual box size=0.028 0.040 0.052; visual cylinder length=0.0875 radius=0.004
Joints:
- joint battery_tray_joint: origin xyz=0.1293 0 0.0305 rpy=0 0 0 -> xyz=0.1003 0 -0.0017 rpy=0 0 0
