Commit message: calib: AprilTag camera extrinsic 2026-07-24 (position RMS 9.6mm)
Re-calibrated base_link->camera_link for the direct-mounted Gemini 2 (the
gimbal-era extrinsic was void). 7 poses (3 arc + 4 line) in a tight room via
new --far-dist/--near-dist collection args; position-only RMS 9.6mm.

- camera_joint: xyz 0.061376 0 0.051154 / rpy 0 -> xyz 0.1017 0.0137 0.0535
  / rpy -0.0171 -0.1196 0.0323 (optical center; z=0.0535 ruler-fixed).
- camera_link visual/collision origin -> -0.0407 -0.0124 0.0023 so the body
  mesh renders at its CAD location while camera_link is the optical center
  (appearance only, separate from the calibration).
- Regenerate ROS URDFs (mentorpi_so101 + viewer) and Isaac URDFs.
- calibrate_camera_extrinsic.py: add --far-dist/--near-dist for tight rooms.

Co-Authored-By: Claude Opus 4.8 <noreply@anthropic.com>

File: isaac/mentorpi.isaac.urdf (robot description, URDF)
Before this commit: robot mentorpi, 11 links, 10 joints
Joints:
- joint camera_joint: origin xyz=0.061376 0 0.051154 rpy=0 0 0 -> xyz=0.1017 0.0137 0.0535 rpy=-0.0171 -0.1196 0.0323

File: isaac/mentorpi_so101.isaac.urdf (robot description, URDF)
Before this commit: robot mentorpi, 22 links, 21 joints
Joints:
- joint camera_joint: origin xyz=0.061376 0 0.051154 rpy=0 0 0 -> xyz=0.1017 0.0137 0.0535 rpy=-0.0171 -0.1196 0.0323

File: src/mentorpi_description/urdf/mecanum.xacro (robot description, xacro)
@@ -96,5 +96,5 @@
     <origin xyz="-0.054 0 0.05" rpy="0 0 0"/>
   </joint>
-  <!-- ===== Camera (external transform pending recalibration) ===== -->
+  <!-- ===== Camera (Gemini 2, AprilTag hand-eye calibrated) ===== -->
   <link name="camera_link">
     <inertial>
@@ -103,15 +103,15 @@
       <inertia ixx="1.44E-05" ixy="0" ixz="0" iyy="1.66E-06" iyz="0" izz="1.46E-05"/>
     </inertial>
-    <!-- 直装方案: 云台已拆除, 相机直接贴装基座、无支撑。camera_link 回归
-         cam_Link.STL 的本体原点(机身顶面中心), 故 visual/collision 偏移归零,
-         与 camera_joint 的 vendor CAD 直装值成对。光学系挂在本体原点上属近似,
-         待 AprilTag 重标精化到真实光学中心。 -->
+    <!-- 视觉修正(纯外观,与标定分离): camera_link 现是 AprilTag 标定的光学中心,
+         而 cam_Link.STL 以机身顶面中心为原点建模。此偏移把网格本体拉回 CAD 本体位
+         (= CAD 本体 0.061376/0/0.051154 减光学中心, 转到 camera_link 帧); 不加则
+         机身网格前移 ~4cm 看似装歪。改标定时按新光学中心重算, 勿手改凑render。 -->
     <visual>
-      <origin rpy="0 0 0" xyz="0 0 0"/>
+      <origin rpy="0 0 0" xyz="-0.0407 -0.0124 0.0023"/>
       <geometry><mesh filename="package://mentorpi_description/meshes/mecanum/cam_Link.STL"/></geometry>
       <material name="black"/>
     </visual>
     <collision>
-      <origin rpy="0 0 0" xyz="0 0 0"/>
+      <origin rpy="0 0 0" xyz="-0.0407 -0.0124 0.0023"/>
       <geometry><mesh filename="package://mentorpi_description/meshes/mecanum/cam_Link.STL"/></geometry>
     </collision>
@@ -120,8 +120,8 @@
     <parent link="base_link"/>
     <child link="camera_link"/>
-    <!-- Vendor CAD 直装值(从 mecanum.pre_calibration.xacro 恢复)。相机直接贴装
-         基座、无支撑; 这是粗定位, 实装可能有位移。最终固定后跑 AprilTag 手眼
-         标定, 用 calibrate_camera_extrinsic.py 的 update-xacro 选项精化本变换。 -->
-    <origin xyz="0.061376 0 0.051154" rpy="0 0 0"/>
+    <!-- AprilTag hand-eye calibration, 2026-07-24 (直装无支撑相机, 光学中心;
+         position-only RMS 9.6mm, 7 poses; z=0.0535 尺量固定, 平面运动不可观)。
+         重标: scripts/calibrate_camera_extrinsic.py 的 update-xacro 选项。 -->
+    <origin xyz="0.1017 0.0137 0.0535" rpy="-0.0171 -0.1196 0.0323"/>
   </joint>
   <!-- Offline preview only; Orbbec owns these frames on hardware. -->

File: src/mentorpi_description/urdf/mentorpi_so101.urdf (robot description, URDF)
Before this commit: robot mentorpi, 22 links, 21 joints
Joints:
- joint camera_joint: origin xyz=0.061376 0 0.051154 rpy=0 0 0 -> xyz=0.1017 0.0137 0.0535 rpy=-0.0171 -0.1196 0.0323

File: src/mentorpi_description/urdf/mentorpi_so101.viewer.urdf (robot description, URDF)
Before this commit: robot mentorpi, 22 links, 21 joints
Joints:
- joint camera_joint: origin xyz=0.061376 0 0.051154 rpy=0 0 0 -> xyz=0.1017 0.0137 0.0535 rpy=-0.0171 -0.1196 0.0323
